File: KiCADProjects/Divisor/Divisor_x8.sch (KiCad schematic (older format))
At the start: 18 parts, among them J1 SMA_Female, J2 SMA_Female, J3 SMA_Female, J4 SMA_Female, J5 SMA_Female, J6 SMA_Female, J7 SMA_Female, J8 SMA_Female, J9 SMA_Female

Commit message: Versión con sys clk a 100 MHz. Archivos de proyecto
Parts:
- R1, R2, R3, R4, R5, R6, R7, R8, R9: value 39 -> 38.8
Changed lines of the file:
@@
 P 4375 3650
 F 0 "R1" V 4275 3650 50  0000 C CNN
-F 1 "39" V 4375 3650 50  0000 C CNN
+F 1 "38.8" V 4375 3650 50  0000 C CNN
 F 2 "Resistor_SMD:R_0805_2012Metric_Pad1.15x1.40mm_HandSolder" V 4305 3650 50  0001 C CNN
 F 3 "~" H 4375 3650 50  0001 C CNN
@@
 P 4900 4900
 F 0 "R5" V 4800 4900 50  0000 C CNN
-F 1 "39" V 4900 4900 50  0000 C CNN
+F 1 "38.8" V 4900 4900 50  0000 C CNN
 F 2 "Resistor_SMD:R_0805_2012Metric_Pad1.15x1.40mm_HandSolder" V 4830 4900 50  0001 C CNN
 F 3 "~" H 4900 4900 50  0001 C CNN
@@
 P 4900 4150
 F 0 "R4" V 4800 4150 50  0000 C CNN
-F 1 "39" V 4900 4150 50  0000 C CNN
+F 1 "38.8" V 4900 4150 50  0000 C CNN
 F 2 "Resistor_SMD:R_0805_2012Metric_Pad1.15x1.40mm_HandSolder" V 4830 4150 50  0001 C CNN
 F 3 "~" H 4900 4150 50  0001 C CNN
@@
 P 4900 3150
 F 0 "R3" V 4800 3150 50  0000 C CNN
-F 1 "39" V 4900 3150 50  0000 C CNN
+F 1 "38.8" V 4900 3150 50  0000 C CNN
 F 2 "Resistor_SMD:R_0805_2012Metric_Pad1.15x1.40mm_HandSolder" V 4830 3150 50  0001 C CNN
 F 3 "~" H 4900 3150 50  0001 C CNN
@@
 P 4900 2400
 F 0 "R2" V 4800 2400 50  0000 C CNN
-F 1 "39" V 4900 2400 50  0000 C CNN
+F 1 "38.8" V 4900 2400 50  0000 C CNN
 F 2 "Resistor_SMD:R_0805_2012Metric_Pad1.15x1.40mm_HandSolder" V 4830 2400 50  0001 C CNN
 F 3 "~" H 4900 2400 50  0001 C CNN
@@
 P 5630 4900
 F 0 "R9" V 5530 4900 50  0000 C CNN
-F 1 "39" V 5630 4900 50  0000 C CNN
+F 1 "38.8" V 5630 4900 50  0000 C CNN
 F 2 "Resistor_SMD:R_0805_2012Metric_Pad1.15x1.40mm_HandSolder" V 5560 4900 50  0001 C CNN
 F 3 "~" H 5630 4900 50  0001 C CNN
@@
 P 5630 4150
 F 0 "R8" V 5530 4150 50  0000 C CNN
-F 1 "39" V 5630 4150 50  0000 C CNN
+F 1 "38.8" V 5630 4150 50  0000 C CNN
 F 2 "Resistor_SMD:R_0805_2012Metric_Pad1.15x1.40mm_HandSolder" V 5560 4150 50  0001 C CNN
 F 3 "~" H 5630 4150 50  0001 C CNN
@@
 P 5630 3150
 F 0 "R7" V 5530 3150 50  0000 C CNN
-F 1 "39" V 5630 3150 50  0000 C CNN
+F 1 "38.8" V 5630 3150 50  0000 C CNN
 F 2 "Resistor_SMD:R_0805_2012Metric_Pad1.15x1.40mm_HandSolder" V 5560 3150 50  0001 C CNN
 F 3 "~" H 5630 3150 50  0001 C CNN
@@
 P 5630 2400
 F 0 "R6" V 5530 2400 50  0000 C CNN
-F 1 "39" V 5630 2400 50  0000 C CNN
+F 1 "38.8" V 5630 2400 50  0000 C CNN
 F 2 "Resistor_SMD:R_0805_2012Metric_Pad1.15x1.40mm_HandSolder" V 5560 2400 50  0001 C CNN
 F 3 "~" H 5630 2400 50  0001 C CNN
